Commit message: Gazebo is fixed, robot appears

File: rover_description/urdf/rover.urdf.xacro (robot description, xacro)
@@ -3,4 +3,5 @@
 <robot name="scarab"
     xmlns:xacro="http://ros.org/wiki/xacro">
+    <xacro:property name="pkg_path" value="$(find rover_description)" />
     <xacro:arg name="is_sim" default="true" />
     <xacro:arg name="is_ignition" default="true"/>
@@ -25,5 +26,5 @@
             <geometry>
                 <!--<box size="1 0.6 0.3"/>-->
-                <mesh filename="package://rover_description/meshes/base_link.stl" scale="0.001 0.001 0.001" />
+                <mesh filename="file://${pkg_path}/meshes/base_link.stl" scale="0.001 0.001 0.001" />
             </geometry>
             <material name="gray">
@@ -34,5 +35,5 @@
             <origin rpy="0 0 1.579795" xyz="0 0 0"/>
             <geometry>
-                <mesh filename="package://rover_description/meshes/base_link.stl" scale="0.001 0.001 0.001" />
+                <mesh filename="file://${pkg_path}/meshes/base_link.stl" scale="0.001 0.001 0.001" />
             </geometry>
         </collision>
@@ -54,14 +55,14 @@
             <origin rpy="0 0 0" xyz="0 0 0"/>
             <geometry>
-                <mesh filename="package://rover_description/meshes/suspension_left_link_a.stl" scale="0.001 0.001 0.001" />
-            </geometry>
-            <material name="yellow">
-                <color rgba="1 1 0 1"/>
-            </material>
-        </visual>
-        <collision>
-            <origin rpy="0 0 0" xyz="0 0 0"/>
-            <geometry>
-                <mesh filename="package://rover_description/meshes/suspension_left_link_a.stl" scale="0.001 0.001 0.001" />
+                <mesh filename="file://${pkg_path}/meshes/suspension_left_link_a.stl" scale="0.001 0.001 0.001" />
+            </geometry>
+            <material name="yellow">
+                <color rgba="1 1 0 1"/>
+            </material>
+        </visual>
+        <collision>
+            <origin rpy="0 0 0" xyz="0 0 0"/>
+            <geometry>
+                <mesh filename="file://${pkg_path}/meshes/suspension_left_link_a.stl" scale="0.001 0.001 0.001" />
             </geometry>
         </collision>
@@ -84,14 +85,14 @@
             <origin rpy="0 0 0" xyz="0 0 0"/>
             <geometry>
-                <mesh filename="package://rover_description/meshes/suspension_left_link_b.stl" scale="0.001 0.001 0.001" />
-            </geometry>
-            <material name="yellow">
-                <color rgba="1 1 0 1"/>
-            </material>
-        </visual>
-        <collision>
-            <origin rpy="0 0 0" xyz="0 0 0"/>
-            <geometry>
-                <mesh filename="package://rover_description/meshes/suspension_left_link_b.stl" scale="0.001 0.001 0.001" />
+                <mesh filename="file://${pkg_path}/meshes/suspension_left_link_b.stl" scale="0.001 0.001 0.001" />
+            </geometry>
+            <material name="yellow">
+                <color rgba="1 1 0 1"/>
+            </material>
+        </visual>
+        <collision>
+            <origin rpy="0 0 0" xyz="0 0 0"/>
+            <geometry>
+                <mesh filename="file://${pkg_path}/meshes/suspension_left_link_b.stl" scale="0.001 0.001 0.001" />
             </geometry>
         </collision>
@@ -115,14 +116,14 @@
             <origin rpy="0 0 0" xyz="0 0 0"/>
             <geometry>
-                <mesh filename="package://rover_description/meshes/suspension_right_link_a.stl" scale="0.001 0.001 0.001" />
-            </geometry>
-            <material name="yellow">
-                <color rgba="1 1 0 1"/>
-            </material>
-        </visual>
-        <collision>
-            <origin rpy="0 0 0" xyz="0 0 0"/>
-            <geometry>
-                <mesh filename="package://rover_description/meshes/suspension_right_link_a.stl" scale="0.001 0.001 0.001" />
+                <mesh filename="file://${pkg_path}/meshes/suspension_right_link_a.stl" scale="0.001 0.001 0.001" />
+            </geometry>
+            <material name="yellow">
+                <color rgba="1 1 0 1"/>
+            </material>
+        </visual>
+        <collision>
+            <origin rpy="0 0 0" xyz="0 0 0"/>
+            <geometry>
+                <mesh filename="file://${pkg_path}/meshes/suspension_right_link_a.stl" scale="0.001 0.001 0.001" />
             </geometry>
         </collision>
@@ -143,14 +144,14 @@
             <origin rpy="0 0 0" xyz="0 0 0"/>
             <geometry>
-                <mesh filename="package://rover_description/meshes/suspension_right_link_b.stl" scale="0.001 0.001 0.001" />
-            </geometry>
-            <material name="yellow">
-                <color rgba="1 1 0 1"/>
-            </material>
-        </visual>
-        <collision>
-            <origin rpy="0 0 0" xyz="0 0 0"/>
-            <geometry>
-                <mesh filename="package://rover_description/meshes/suspension_right_link_b.stl" scale="0.001 0.001 0.001" />
+                <mesh filename="file://${pkg_path}/meshes/suspension_right_link_b.stl" scale="0.001 0.001 0.001" />
+            </geometry>
+            <material name="yellow">
+                <color rgba="1 1 0 1"/>
+            </material>
+        </visual>
+        <collision>
+            <origin rpy="0 0 0" xyz="0 0 0"/>
+            <geometry>
+                <mesh filename="file://${pkg_path}/meshes/suspension_right_link_b.stl" scale="0.001 0.001 0.001" />
             </geometry>
         </collision>
