Commit message: Added colour to rover model

File: rover_description/urdf/Final.xacro (robot description, xacro)
@@ -15,5 +15,7 @@
       <mesh filename="package://rover_description/meshes/base_link.stl" scale="0.001 0.001 0.001"/>
     </geometry>
-    <material name="silver"/>
+    <material name="nice_navy">
+        <color rgba="0.12 0.18 0.4 1"/>
+    </material>
   </visual>
   <collision>
@@ -35,5 +37,7 @@
       <mesh filename="package://rover_description/meshes/Wheel2_1.stl" scale="0.001 0.001 0.001"/>
     </geometry>
-    <material name="silver"/>
+    <material name="black">
+        <color rgba="0.01 0.01 0.01 1"/>
+    </material>
   </visual>
   <collision>
@@ -55,5 +59,7 @@
       <mesh filename="package://rover_description/meshes/Wheel1_1.stl" scale="0.001 0.001 0.001"/>
     </geometry>
-    <material name="silver"/>
+    <material name="black">
+        <color rgba="0.01 0.01 0.01 1"/>
+    </material>
   </visual>
   <collision>
@@ -75,5 +81,7 @@
       <mesh filename="package://rover_description/meshes/Wheel2__1__2.stl" scale="0.001 0.001 0.001"/>
     </geometry>
-    <material name="silver"/>
+    <material name="black">
+        <color rgba="0.01 0.01 0.01 1"/>
+    </material>
   </visual>
   <collision>
@@ -95,5 +103,7 @@
       <mesh filename="package://rover_description/meshes/Wheel2__1__1.stl" scale="0.001 0.001 0.001"/>
     </geometry>
-    <material name="silver"/>
+    <material name="black">
+        <color rgba="0.01 0.01 0.01 1"/>
+    </material>
   </visual>
   <collision>
@@ -115,5 +125,7 @@
       <mesh filename="package://rover_description/meshes/Side1_1.stl" scale="0.001 0.001 0.001"/>
     </geometry>
-    <material name="silver"/>
+    <material name="soft_orange">
+        <color rgba="0.85 0.45 0.15 1"/>
+    </material>
   </visual>
   <collision>
@@ -135,5 +147,7 @@
       <mesh filename="package://rover_description/meshes/Side2_1.stl" scale="0.001 0.001 0.001"/>
     </geometry>
-    <material name="silver"/>
+    <material name="soft_orange">
+        <color rgba="0.85 0.45 0.15 1"/>
+    </material>
   </visual>
   <collision>

Commit message: fixed final xacro file w vasee and rid

File: rover_description/urdf/Final.xacro (robot description, xacro)
@@ -7,5 +7,5 @@
   <inertial>
     <origin xyz="0.23371470080552523 0.3424215459495483 0.11792924666461195" rpy="0 0 0"/>
-    <mass value="570.3291503802121"/>
+    <mass value="36.0"/>
     <inertia ixx="28.457355" iyy="14.276737" izz="34.968035" ixy="0.085086" iyz="0.387247" ixz="-0.119086"/>
   </inertial>
@@ -29,5 +29,5 @@
   <inertial>
     <origin xyz="0.060000000000048695 9.626243984289795e-07 0.00010157518963996304" rpy="0 0 0"/>
-    <mass value="22.44587224692876"/>
+    <mass value="3.5"/>
     <inertia ixx="0.234154" iyy="0.134117" izz="0.153907" ixy="-0.0" iyz="8e-06" ixz="0.0"/>
   </inertial>
@@ -51,5 +51,5 @@
   <inertial>
     <origin xyz="0.05999999999997653 1.1249441103089453e-06 0.00010186480729457159" rpy="0 0 0"/>
-    <mass value="22.445872246928765"/>
+    <mass value="3.5"/>
     <inertia ixx="0.234154" iyy="0.134117" izz="0.153907" ixy="-0.0" iyz="8e-06" ixz="0.0"/>
   </inertial>
@@ -73,5 +73,5 @@
   <inertial>
     <origin xyz="-0.059999999999952314 1.1891813821787722e-06 0.00010132422446335054" rpy="0 0 0"/>
-    <mass value="22.445872246928758"/>
+    <mass value="3.5"/>
     <inertia ixx="0.234154" iyy="0.134117" izz="0.153907" ixy="0.0" iyz="8e-06" ixz="-0.0"/>
   </inertial>
@@ -95,5 +95,5 @@
   <inertial>
     <origin xyz="-0.7537999999999477 7.512494407269088e-05 0.00026586480728614525" rpy="0 0 0"/>
-    <mass value="22.445872246928758"/>
+    <mass value="3.5"/>
     <inertia ixx="0.234154" iyy="0.134117" izz="0.153907" ixy="0.0" iyz="8e-06" ixz="-0.0"/>
   </inertial>
@@ -117,5 +117,5 @@
   <inertial>
     <origin xyz="-0.04997257661493937 0.0004804691908492642 0.02785086678998311" rpy="0 0 0"/>
-    <mass value="48.074770975371656"/>
+    <mass value="5.0"/>
     <inertia ixx="3.901891" iyy="0.088961" izz="3.911318" ixy="-0.000394" iyz="0.044008" ixz="4.1e-05"/>
   </inertial>
@@ -139,5 +139,5 @@
   <inertial>
     <origin xyz="0.050023043717073556 0.00048164194190997156 0.028033001206298203" rpy="0 0 0"/>
-    <mass value="48.07477097518222"/>
+    <mass value="5.0"/>
     <inertia ixx="3.900293" iyy="0.087383" izz="3.911242" ixy="-0.000484" iyz="0.047745" ixz="2.8e-05"/>
   </inertial>
@@ -182,5 +182,5 @@
   <axis xyz="1.0 -0.0 0.0"/>
 </joint>
-<joint name="Revolute 18" type="continuous">
+<joint name="Revolute 18" type="fixed">
   <origin xyz="0.63 0.37785 0.1081" rpy="0 0 0"/>
   <parent link="base_link"/>
@@ -188,5 +188,5 @@
   <axis xyz="1.0 -0.0 0.0"/>
 </joint>
-<joint name="Revolute 19" type="continuous">
+<joint name="Revolute 19" type="fixed">
   <origin xyz="-0.1638 0.37785 0.1081" rpy="0 0 0"/>
   <parent link="base_link"/>
