Commit message: Adding Final files from urdf
adding four files from rover_description/urdf from 'newRobotModel' branch to the main branch

File: src/rover_description/urdf/materials.xacro (robot description, xacro)
@@ -1,28 +1,6 @@
-<?xml version="1.0" encoding="utf-8"?>
-<robot name="materials"
-  xmlns:xacro="http://ros.org/wiki/xacro">
-  <material name="black">
-    <color rgba="0.1 0.1 0.1 1.0" />
-  </material>
-  <material name="blue">
-    <color rgba="0.0 0.0 0.8 1.0" />
-  </material>
-  <material name="green">
-    <color rgba="0.4 0.9 0.4 1.0" />
-  </material>
-  <material name="gray">
-    <color rgba="0.7 0.7 0.7 1.0" />
-  </material>
-  <material name="darkgray">
-    <color rgba="0.3 0.3 0.3 1.0" />
-  </material>
-  <material name="red">
-    <color rgba="0.8 0.0 0.0 1.0" />
-  </material>
-  <material name="white">
-    <color rgba="1.0 1.0 1.0 1.0" />
-  </material>
-  <material name="yellow">
-    <color rgba="0.8 0.8 0.0 1.0" />
-  </material>
+<?xml version="1.0" ?>
+<robot name="Final" xmlns:xacro="http://www.ros.org/wiki/xacro" >
+<material name="silver">
+  <color rgba="0.700 0.700 0.700 1.000"/>
+</material>
 </robot>
