Commit message: fixed rviz issues!

File: src/rover_description/urdf/Final.xacro (robot description, xacro)
@@ -4,4 +4,12 @@
 <xacro:include filename="$(find rover_description)/urdf/Final.trans" />
 <xacro:include filename="$(find rover_description)/urdf/Final.gazebo" />
+<xacro:arg name="is_ignition" default="true"/>
+<xacro:include filename="$(find rover_description)/urdf/rover_control.xacro" />
+<link name="base_footprint"/>
+<joint name="base_footprint_joint" type="fixed">
+  <parent link="base_footprint"/>
+  <child link="base_link"/>
+  <origin xyz="0 0 0.393" rpy="0 0 0"/>
+</joint>
 <link name="base_link">
   <inertial>

Commit message: rviz fixed, slam working, controller rover works, weight of rover has been adjusted by a factor of 10

File: src/rover_description/urdf/Final.xacro (robot description, xacro)
@@ -4,4 +4,5 @@
 <xacro:include filename="$(find rover_description)/urdf/Final.trans" />
 <xacro:include filename="$(find rover_description)/urdf/Final.gazebo" />
+<xacro:include filename="$(find rover_description)/urdf/sensors/lidar3d.xacro" />
 <xacro:arg name="is_ignition" default="true"/>
 <xacro:include filename="$(find rover_description)/urdf/rover_control.xacro" />
@@ -15,5 +16,5 @@
   <inertial>
     <origin xyz="0.23371470080552523 0.3424215459495483 0.11792924666461195" rpy="0 0 0"/>
-    <mass value="36.0"/>
+    <mass value="360.0"/>
     <inertia ixx="28.457355" iyy="14.276737" izz="34.968035" ixy="0.085086" iyz="0.387247" ixz="-0.119086"/>
   </inertial>
@@ -37,5 +38,5 @@
   <inertial>
     <origin xyz="0.060000000000048695 9.626243984289795e-07 0.00010157518963996304" rpy="0 0 0"/>
-    <mass value="3.5"/>
+    <mass value="35.0"/>
     <inertia ixx="0.234154" iyy="0.134117" izz="0.153907" ixy="-0.0" iyz="8e-06" ixz="0.0"/>
   </inertial>
@@ -59,5 +60,5 @@
   <inertial>
     <origin xyz="0.05999999999997653 1.1249441103089453e-06 0.00010186480729457159" rpy="0 0 0"/>
-    <mass value="3.5"/>
+    <mass value="35.0"/>
     <inertia ixx="0.234154" iyy="0.134117" izz="0.153907" ixy="-0.0" iyz="8e-06" ixz="0.0"/>
   </inertial>
@@ -81,5 +82,5 @@
   <inertial>
     <origin xyz="-0.059999999999952314 1.1891813821787722e-06 0.00010132422446335054" rpy="0 0 0"/>
-    <mass value="3.5"/>
+    <mass value="35.0"/>
     <inertia ixx="0.234154" iyy="0.134117" izz="0.153907" ixy="0.0" iyz="8e-06" ixz="-0.0"/>
   </inertial>
@@ -103,5 +104,5 @@
   <inertial>
     <origin xyz="-0.7537999999999477 7.512494407269088e-05 0.00026586480728614525" rpy="0 0 0"/>
-    <mass value="3.5"/>
+    <mass value="35.0"/>
     <inertia ixx="0.234154" iyy="0.134117" izz="0.153907" ixy="0.0" iyz="8e-06" ixz="-0.0"/>
   </inertial>
@@ -125,5 +126,5 @@
   <inertial>
     <origin xyz="-0.04997257661493937 0.0004804691908492642 0.02785086678998311" rpy="0 0 0"/>
-    <mass value="5.0"/>
+    <mass value="50.0"/>
     <inertia ixx="3.901891" iyy="0.088961" izz="3.911318" ixy="-0.000394" iyz="0.044008" ixz="4.1e-05"/>
   </inertial>
@@ -147,5 +148,5 @@
   <inertial>
     <origin xyz="0.050023043717073556 0.00048164194190997156 0.028033001206298203" rpy="0 0 0"/>
-    <mass value="5.0"/>
+    <mass value="50.0"/>
     <inertia ixx="3.900293" iyy="0.087383" izz="3.911242" ixy="-0.000484" iyz="0.047745" ixz="2.8e-05"/>
   </inertial>
