Commit message: rename rover urdf files

File: src/rover_description/urdf/rover.control.xacro (robot description, xacro)
@@ -1,17 +1,8 @@
 <?xml version="1.0"?>
-<robot name="Final"
-xmlns:xacro="http://ros.org/wiki/xacro">
+<robot name="Deimos/control" xmlns:xacro="http://ros.org/wiki/xacro">
   <ros2_control name="GazeboSystem" type="system">
-    <xacro:if value="$(arg is_ignition)">
-      <hardware>
-        <plugin>ign_ros2_control/IgnitionSystem</plugin>
-      </hardware>
-    </xacro:if>
-    <!-- ROS 2 Iron or above -->
-    <xacro:unless value="$(arg is_ignition)">
-      <hardware>
-        <plugin>gz_ros2_control/GazeboSimSystem</plugin>
-      </hardware>
-    </xacro:unless>
+    <hardware>
+      <plugin>ign_ros2_control/IgnitionSystem</plugin>
+    </hardware>
     <!-- Revolute 14: front wheel on Side2_1 (left side) -->
     <joint name="Revolute 14">
@@ -50,5 +41,4 @@
       <state_interface name="velocity" />
     </joint>
-    <!-- Revolute 18 and 19 are fixed joints — no control interfaces needed -->
   </ros2_control>
 </robot>

File: src/rover_description/urdf/rover.gazebo.xacro (robot description, xacro)
@@ -1,4 +1,4 @@
 <?xml version="1.0" ?>
-<robot name="Final" xmlns:xacro="http://www.ros.org/wiki/xacro" >
+<robot name="Deimos/gazebo" xmlns:xacro="http://www.ros.org/wiki/xacro" >
 <xacro:property name="body_color" value="Gazebo/Silver" />
 <gazebo>

File: src/rover_description/urdf/rover.urdf.xacro (robot description, xacro)
@@ -1,352 +1,211 @@
 <?xml version="1.0"?>
-<!--    http://wiki.ros.org/urdf/XML/link   -->
-<robot name="scarab"
-    xmlns:xacro="http://ros.org/wiki/xacro">
-    <xacro:arg name="is_sim" default="true" />
-    <xacro:arg name="is_ignition" default="true"/>
-    <xacro:include filename="$(find rover_description)/urdf/rover_gazebo.xacro" />
-    <xacro:include filename="$(find rover_description)/urdf/rover_control.xacro" />
-    <xacro:include filename="$(find rover_description)/urdf/sensors/realsense.xacro" />
-    <xacro:include filename="$(find rover_description)/urdf/sensors/lidar3d.xacro" />
-    <link name="base_footprint"/>
-    <joint name="base_footprint_joint" type="fixed">
-        <parent link="base_footprint"/>
-        <child link="base_link"/>
-        <origin xyz="0 0 0.393" rpy="0 0 3.14159"/>
-    </joint>
-    <!-- This is the body of the rover -->
-    <link name="base_link">
-        <inertial>
-            <origin xyz="0 0 0" rpy="0 0 0"/>
-            <mass value="15.0"/>
-            <inertia ixx="0.5" ixy="0.0" ixz="0.0" iyy="0.7" iyz="0.0" izz="1.0"/>
-        </inertial>
-        <visual>
-            <origin rpy="0 0 1.579795" xyz="0 0 0"/>
-            <geometry>
-                <!--<box size="1 0.6 0.3"/>-->
-                <mesh filename="package://rover_description/meshes/base_link.stl" scale="0.001 0.001 0.001" />
-            </geometry>
-            <material name="gray">
-                <color rgba="0.4 0.4 0.4 1"/>
-            </material>
-        </visual>
-        <collision>
-            <origin rpy="0 0 1.579795" xyz="0 0 0"/>
-            <geometry>
-                <mesh filename="package://rover_description/meshes/base_link.stl" scale="0.001 0.001 0.001" />
-            </geometry>
-        </collision>
-    </link>
-    <!-- This is the left suspension assembly -->
-    <joint name="susLeft_joint" type="fixed">
-        <parent link="base_link" />
-        <child link="susLeft_link" />
-        <origin xyz ="-0.1 -0.239 0.04" rpy="0 0 -1.579795" />
-        <axis xyz="1 0 0" />
-    </joint>
-    <link name="susLeft_link">
-        <inertial>
-            <origin xyz="0 0 0" rpy="0 0 0"/>
-            <mass value="2.0"/>
-            <inertia ixx="0.1" ixy="0.0" ixz="0.0" iyy="0.1" iyz="0.0" izz="0.1"/>
-        </inertial>
-        <visual>
-            <origin rpy="0 0 0" xyz="0 0 0"/>
-            <geometry>
-                <mesh filename="package://rover_description/meshes/suspension_left_link_a.stl" scale="0.001 0.001 0.001" />
-            </geometry>
-            <material name="yellow">
-                <color rgba="1 1 0 1"/>
-            </material>
-        </visual>
-        <collision>
-            <origin rpy="0 0 0" xyz="0 0 0"/>
-            <geometry>
-                <mesh filename="package://rover_description/meshes/suspension_left_link_a.stl" scale="0.001 0.001 0.001" />
-            </geometry>
-        </collision>
-    </link>
-    <joint name="susLeft_joint_b" type="continuous">
-        <parent link="susLeft_link" />
-        <child link="susLeft_link_b" />
-        <origin xyz ="0.052 -0.156485 -0.088953" rpy="0 0 0" />
-        <axis xyz="1 0 0" />
-        <dynamics damping="0.1" friction="0.1"/>
-        <limit effort="50" velocity="1"/>
-    </joint>
-    <link name="susLeft_link_b">
-        <inertial>
-            <origin xyz="0 0 0" rpy="0 0 0"/>
-            <mass value="2.0"/>
-            <inertia ixx="0.1" ixy="0.0" ixz="0.0" iyy="0.1" iyz="0.0" izz="0.1"/>
-        </inertial>
-        <visual>
-            <origin rpy="0 0 0" xyz="0 0 0"/>
-            <geometry>
-                <mesh filename="package://rover_description/meshes/suspension_left_link_b.stl" scale="0.001 0.001 0.001" />
-            </geometry>
-            <material name="yellow">
-                <color rgba="1 1 0 1"/>
-            </material>
-        </visual>
-        <collision>
-            <origin rpy="0 0 0" xyz="0 0 0"/>
-            <geometry>
-                <mesh filename="package://rover_description/meshes/suspension_left_link_b.stl" scale="0.001 0.001 0.001" />
-            </geometry>
-        </collision>
-    </link>
-    <!-- This is the right suspension assembly -->
-    <joint name="susRight_joint" type="fixed">
-        <parent link="base_link" />
-        <child link="susRight_link" />
-        <origin xyz ="-0.1 0.21 0.04" rpy="0 0 -1.579795" />
-        <axis xyz="1 0 0" />
-        <dynamics damping="0.1" friction="0.1"/>
-        <limit effort="50" velocity="1"/>
-    </joint>
-    <link name="susRight_link">
-        <inertial>
-            <origin xyz="0 0 0" rpy="0 0 0"/>
-            <mass value="2.0"/>
-            <inertia ixx="0.1" ixy="0.0" ixz="0.0" iyy="0.1" iyz="0.0" izz="0.1"/>
-        </inertial>
-        <visual>
-            <origin rpy="0 0 0" xyz="0 0 0"/>
-            <geometry>
-                <mesh filename="package://rover_description/meshes/suspension_right_link_a.stl" scale="0.001 0.001 0.001" />
-            </geometry>
-            <material name="yellow">
-                <color rgba="1 1 0 1"/>
-            </material>
-        </visual>
-        <collision>
-            <origin rpy="0 0 0" xyz="0 0 0"/>
-            <geometry>
-                <mesh filename="package://rover_description/meshes/suspension_right_link_a.stl" scale="0.001 0.001 0.001" />
-            </geometry>
-        </collision>
-    </link>
-    <joint name="susRight_joint_b" type="continuous">
-        <parent link="susRight_link" />
-        <child link="susRight_link_b" />
-        <origin xyz ="-0.038 -0.156485 -0.088953" rpy="0 0 0" />
-        <axis xyz="1 0 0" />
-    </joint>
-    <link name="susRight_link_b">
-        <inertial>
-            <origin xyz="0 0 0" rpy="0 0 0"/>
-            <mass value="2.0"/>
-            <inertia ixx="0.1" ixy="0.0" ixz="0.0" iyy="0.1" iyz="0.0" izz="0.1"/>
-        </inertial>
-        <visual>
-            <origin rpy="0 0 0" xyz="0 0 0"/>
-            <geometry>
-                <mesh filename="package://rover_description/meshes/suspension_right_link_b.stl" scale="0.001 0.001 0.001" />
-            </geometry>
-            <material name="yellow">
-                <color rgba="1 1 0 1"/>
-            </material>
-        </visual>
-        <collision>
-            <origin rpy="0 0 0" xyz="0 0 0"/>
-            <geometry>
-                <mesh filename="package://rover_description/meshes/suspension_right_link_b.stl" scale="0.001 0.001 0.001" />
-            </geometry>
-        </collision>
-    </link>
-    <!-- This is the front right wheel of the rover -->
-    <joint name="wheel1_joint" type="continuous">
-        <parent link="susRight_link_b" />
-        <child link="wheel1_link" />
-        <origin xyz ="-0.05 -0.20796 -0.196506" rpy="0 0 0" />
-        <axis xyz="1 0 0" />
-    </joint>
-    <link name="wheel1_link">
-        <inertial>
-            <origin xyz="0 0 0" rpy="0 0 0"/>
-            <mass value="1.0"/>
-            <inertia ixx="0.002" ixy="0.0" ixz="0.0" iyy="0.002" iyz="0.0" izz="0.004"/>
-        </inertial>
-        <visual>
-            <origin rpy="1.579795 0 1.579795" xyz="0 0 0"/>
-            <geometry>
-                <cylinder radius="0.1175" length="0.12"/>
-            </geometry>
-            <material name="black">
-                <color rgba="0.01 0.01 0.01 1"/>
-            </material>
-        </visual>
-        <collision>
-            <origin rpy="1.579795 0 1.579795" xyz="0 0 0"/>
-            <geometry>
-                <cylinder radius="0.1175" length="0.12"/>
-            </geometry>
-        </collision>
-    </link>
-    <!-- This is the front left wheel of the rover -->
-    <joint name="wheel2_joint" type="continuous">
-        <parent link="susLeft_link_b" />
-        <child link="wheel2_link" />
-        <origin xyz ="0.05 -0.20796 -0.196506" rpy="0 0 0" />
-        <axis xyz="1 0 0" />
-    </joint>
-    <link name="wheel2_link">
-        <inertial>
-            <origin xyz="0 0 0" rpy="0 0 0"/>
-            <mass value="1.0"/>
-            <inertia ixx="0.002" ixy="0.0" ixz="0.0" iyy="0.002" iyz="0.0" izz="0.004"/>
-        </inertial>
-        <visual>
-            <origin rpy="1.579795 0 1.579795" xyz="0 0 0"/>
-            <geometry>
-                <cylinder radius="0.1175" length="0.12"/>
-            </geometry>
-            <material name="black">
-                <color rgba="0.01 0.01 0.01 1"/>
-            </material>
-        </visual>
-        <collision>
-            <origin rpy="1.579795 0 1.579795" xyz="0 0 0"/>
-            <geometry>
-                <cylinder radius="0.1175" length="0.12"/>
-            </geometry>
-        </collision>
-    </link>
-    <!-- This is the middle right wheel of the rover -->
-    <joint name="wheel3_joint" type="continuous">
-        <parent link="susRight_link_b" />
-        <child link="wheel3_link" />
-        <origin xyz ="-0.11 0.168268 -0.211155" rpy="0 0 0" />
-        <axis xyz="1 0 0" />
-    </joint>
-    <link name="wheel3_link">
-        <inertial>
-            <origin xyz="0 0 0" rpy="0 0 0"/>
-            <mass value="1.0"/>
-            <inertia ixx="0.002" ixy="0.0" ixz="0.0" iyy="0.002" iyz="0.0" izz="0.004"/>
-        </inertial>
-        <visual>
-            <origin rpy="1.579795 0 1.579795" xyz="0 0 0"/>
-            <geometry>
-                <cylinder radius="0.1175" length="0.12"/>
-            </geometry>
-            <material name="black">
-                <color rgba="0.01 0.01 0.01 1"/>
-            </material>
-        </visual>
-        <collision>
-            <origin rpy="1.579795 0 1.579795" xyz="0 0 0"/>
-            <geometry>
-                <cylinder radius="0.1175" length="0.12"/>
-            </geometry>
-        </collision>
-    </link>
-    <!-- This is the middle left wheel of the rover -->
-    <joint name="wheel4_joint" type="continuous">
-        <parent link="susLeft_link_b" />
-        <child link="wheel4_link" />
-        <origin xyz ="0.1 0.168268 -0.211155" rpy="0 0 0" />
-        <axis xyz="1 0 0" />
-    </joint>
-    <link name="wheel4_link">
-        <inertial>
-            <origin xyz="0 0 0" rpy="0 0 0"/>
-            <mass value="1.0"/>
-            <inertia ixx="0.002" ixy="0.0" ixz="0.0" iyy="0.002" iyz="0.0" izz="0.004"/>
-        </inertial>
-        <visual>
-            <origin rpy="1.579795 0 1.579795" xyz="0 0 0"/>
-            <geometry>
-                <cylinder radius="0.1175" length="0.12"/>
-            </geometry>
-            <material name="black">
-                <color rgba="0.01 0.01 0.01 1"/>
-            </material>
-        </visual>
-        <collision>
-            <origin rpy="1.579795 0 1.579795" xyz="0 0 0"/>
-            <geometry>
-                <cylinder radius="0.1175" length="0.12"/>
-            </geometry>
-        </collision>
-    </link>
-    <!-- This is the back right wheel of the rover -->
-    <joint name="wheel5_joint" type="continuous">
-        <parent link="susRight_link" />
-        <child link="wheel5_link" />
-        <origin xyz ="-0.05 0.35 -0.3" rpy="0 0 0" />
-        <axis xyz="1 0 0" />
-    </joint>
-    <link name="wheel5_link">
-        <inertial>
-            <origin xyz="0 0 0" rpy="0 0 0"/>
-            <mass value="1.0"/>
-            <inertia ixx="0.002" ixy="0.0" ixz="0.0" iyy="0.002" iyz="0.0" izz="0.004"/>
-        </inertial>
-        <visual>
-            <origin rpy="1.579795 0 1.579795" xyz="0 0 0"/>
-            <geometry>
-                <cylinder radius="0.1175" length="0.12"/>
-            </geometry>
-            <material name="black">
-                <color rgba="0.01 0.01 0.01 1"/>
-            </material>
-        </visual>
-        <collision>
-            <origin rpy="1.579795 0 1.579795" xyz="0 0 0"/>
-            <geometry>
-                <cylinder radius="0.1175" length="0.12"/>
-            </geometry>
-        </collision>
-    </link>
-    <!-- This is the back left wheel of the rover -->
-    <joint name="wheel6_joint" type="continuous">
-        <parent link="susLeft_link" />
-        <child link="wheel6_link" />
-        <origin xyz ="0.02 0.35 -0.3" rpy="0 0 0" />
-        <axis xyz="1 0 0" />
-    </joint>
-    <link name="wheel6_link">
-        <inertial>
-            <origin xyz="0 0 0" rpy="0 0 0"/>
-            <mass value="1.0"/>
-            <inertia ixx="0.002" ixy="0.0" ixz="0.0" iyy="0.002" iyz="0.0" izz="0.004"/>
-        </inertial>
-        <visual>
-            <origin rpy="1.579795 0 1.579795" xyz="0 0 0"/>
-            <geometry>
-                <cylinder radius="0.1175" length="0.12"/>
-            </geometry>
-            <material name="black">
-                <color rgba="0.01 0.01 0.01 1"/>
-            </material>
-        </visual>
-        <collision>
-            <origin rpy="1.579795 0 1.579795" xyz="0 0 0"/>
-            <geometry>
-                <cylinder radius="0.1175" length="0.12"/>
-            </geometry>
-        </collision>
-    </link>
-    <!-- This is the back left wheel of the rover
-    <joint name="wheel2_joint" type="continuous">
-        <parent link="base_link" />
-        <child link="wheel2_link" />
-        <origin xyz ="-0.3 0.35 -0.1" rpy="0 0 0" />
-        <axis xyz="0 1 0" />
-    </joint>
-    <link name="wheel2_link">
-        <visual>
-            <origin rpy="1.579795 0 0" xyz="0 0 0"/>
-            <geometry>
-                <cylinder radius="0.15" length="0.1"/>
-            </geometry>
-            <material name="yellow">
-                <color rgba="1 1 0 1"/>
-            </material>
-        </visual>
-    </link>
-     -->
+<robot name="Deimos" xmlns:xacro="http://www.ros.org/wiki/xacro">
+  <xacro:property name="PI" value="3.141592653589793"/>
+  <xacro:include filename="$(find rover_description)/urdf/rover.material.xacro" />
+  <xacro:include filename="$(find rover_description)/urdf/rover.gazebo.xacro" />
+  <xacro:include filename="$(find rover_description)/urdf/sensors/lidar3d.xacro" />
+  <xacro:include filename="$(find rover_description)/urdf/rover.control.xacro" />
+  <link name="base_footprint" />
+  <joint name="base_footprint_joint" type="fixed">
+    <parent link="base_footprint" />
+    <child link="base_link" />
+    <origin xyz="0 0 0" rpy="0 0 ${PI/2}" />
+  </joint>
+  <link name="base_link">
+    <inertial>
+      <origin xyz="0.23371470080552523 0.3424215459495483 0.11792924666461195" rpy="0 0 0" />
+      <mass value="360.0" />
+      <inertia ixx="28.457355" iyy="14.276737" izz="34.968035" ixy="0.085086" iyz="0.387247"
+        ixz="-0.119086" />
+    </inertial>
+    <visual>
+      <origin xyz="0 0 0" rpy="0 0 0" />
+      <geometry>
+        <mesh filename="package://rover_description/meshes/base_link.stl" scale="0.001 0.001 0.001" />
+      </geometry>
+      <material name="nice_navy">
+        <color rgba="0.12 0.18 0.4 1" />
+      </material>
+    </visual>
+    <collision>
+      <origin xyz="0 0 0" rpy="0 0 0" />
+      <geometry>
+        <mesh filename="package://rover_description/meshes/base_link.stl" scale="0.001 0.001 0.001" />
+      </geometry>
+    </collision>
+  </link>
+  <link name="Wheel2_1">
+    <inertial>
+      <origin xyz="0.060000000000048695 9.626243984289795e-07 0.00010157518963996304" rpy="0 0 0" />
+      <mass value="35.0" />
+      <inertia ixx="0.234154" iyy="0.134117" izz="0.153907" ixy="-0.0" iyz="8e-06" ixz="0.0" />
+    </inertial>
+    <visual>
+      <origin xyz="0.1758 0.049434 0.072191" rpy="0 0 0" />
+      <geometry>
+        <mesh filename="package://rover_description/meshes/Wheel2_1.stl" scale="0.001 0.001 0.001" />
+      </geometry>
+      <material name="black">
+        <color rgba="0.01 0.01 0.01 1" />
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