Commit message: refactor urdf xacro

File: src/rover_description/urdf/rover.control.xacro (robot description, xacro)
@@ -1,44 +1,24 @@
 <?xml version="1.0"?>
 <robot name="Deimos/control" xmlns:xacro="http://ros.org/wiki/xacro">
+  <xacro:property name="wheel_min_vel" value="-0.7" />
+  <xacro:property name="wheel_max_vel" value="0.7" />
+  <xacro:macro name="wheel_ros2_control_joint" params="joint_name">
+    <joint name="${joint_name}">
+      <command_interface name="velocity">
+        <param name="min">${wheel_min_vel}</param>
+        <param name="max">${wheel_max_vel}</param>
+      </command_interface>
+      <state_interface name="position" />
+      <state_interface name="velocity" />
+    </joint>
+  </xacro:macro>
   <ros2_control name="GazeboSystem" type="system">
     <hardware>
       <plugin>ign_ros2_control/IgnitionSystem</plugin>
     </hardware>
-    <!-- Revolute 14: front wheel on Side2_1 (left side) -->
-    <joint name="Revolute 14">
-      <command_interface name="velocity">
-        <param name="min">-0.7</param>
-        <param name="max">0.7</param>
-      </command_interface>
-      <state_interface name="position" />
-      <state_interface name="velocity" />
-    </joint>
-    <!-- Revolute 15: rear wheel on Side2_1 (left side) -->
-    <joint name="Revolute 15">
-      <command_interface name="velocity">
-        <param name="min">-0.7</param>
-        <param name="max">0.7</param>
-      </command_interface>
-      <state_interface name="position" />
-      <state_interface name="velocity" />
-    </joint>
-    <!-- Revolute 16: front wheel on Side1_1 (right side) -->
-    <joint name="Revolute 16">
-      <command_interface name="velocity">
-        <param name="min">-0.7</param>
-        <param name="max">0.7</param>
-      </command_interface>
-      <state_interface name="position" />
-      <state_interface name="velocity" />
-    </joint>
-    <!-- Revolute 17: rear wheel on Side1_1 (right side) -->
-    <joint name="Revolute 17">
-      <command_interface name="velocity">
-        <param name="min">-0.7</param>
-        <param name="max">0.7</param>
-      </command_interface>
-      <state_interface name="position" />
-      <state_interface name="velocity" />
-    </joint>
+    <xacro:wheel_ros2_control_joint joint_name="wheel_back_left_joint" />
+    <xacro:wheel_ros2_control_joint joint_name="wheel_front_left_joint" />
+    <xacro:wheel_ros2_control_joint joint_name="wheel_back_right_joint" />
+    <xacro:wheel_ros2_control_joint joint_name="wheel_front_right_joint" />
   </ros2_control>
 </robot>

File: src/rover_description/urdf/rover.gazebo.xacro (robot description, xacro)
@@ -1,53 +1,31 @@
-<?xml version="1.0" ?>
-<robot name="Deimos/gazebo" xmlns:xacro="http://www.ros.org/wiki/xacro" >
-<xacro:property name="body_color" value="Gazebo/Silver" />
-<gazebo>
-  <plugin filename="ign_ros2_control-system"
-          name="ign_ros2_control::IgnitionROS2ControlPlugin">
-    <parameters>$(find rover_controller)/config/controller.yaml</parameters>
-  </plugin>
-</gazebo>
-<gazebo reference="base_link">
-  <material>${body_color}</material>
-  <mu1>0.2</mu1>
-  <mu2>0.2</mu2>
-  <selfCollide>true</selfCollide>
-  <gravity>true</gravity>
-</gazebo>
-<gazebo reference="Wheel2_1">
-  <material>${body_color}</material>
-  <mu1>0.2</mu1>
-  <mu2>0.2</mu2>
-  <selfCollide>true</selfCollide>
-</gazebo>
-<gazebo reference="Wheel1_1">
-  <material>${body_color}</material>
-  <mu1>0.2</mu1>
-  <mu2>0.2</mu2>
-  <selfCollide>true</selfCollide>
-</gazebo>
-<gazebo reference="Wheel2__1__2">
-  <material>${body_color}</material>
-  <mu1>0.2</mu1>
-  <mu2>0.2</mu2>
-  <selfCollide>true</selfCollide>
-</gazebo>
-<gazebo reference="Wheel2__1__1">
-  <material>${body_color}</material>
-  <mu1>0.2</mu1>
-  <mu2>0.2</mu2>
-  <selfCollide>true</selfCollide>
-</gazebo>
-<gazebo reference="Side1_1">
-  <material>${body_color}</material>
-  <mu1>0.2</mu1>
-  <mu2>0.2</mu2>
-  <selfCollide>true</selfCollide>
-</gazebo>
-<gazebo reference="Side2_1">
-  <material>${body_color}</material>
-  <mu1>0.2</mu1>
-  <mu2>0.2</mu2>
-  <selfCollide>true</selfCollide>
-</gazebo>
+<?xml version="1.0"?>
+<robot name="Deimos/gazebo" xmlns:xacro="http://www.ros.org/wiki/xacro">
+  <xacro:property name="body_color" value="Gazebo/Silver" />
+  <xacro:property name="default_mu1" value="0.2" />
+  <xacro:property name="default_mu2" value="0.2" />
+  <xacro:macro name="gazebo_surface" params="link_name">
+    <gazebo reference="${link_name}">
+      <material>${body_color}</material>
+      <mu1>${default_mu1}</mu1>
+      <mu2>${default_mu2}</mu2>
+      <selfCollide>true</selfCollide>
+    </gazebo>
+  </xacro:macro>
+  <!-- ros2_control plugin -->
+  <gazebo>
+    <plugin filename="ign_ros2_control-system"
+      name="ign_ros2_control::IgnitionROS2ControlPlugin">
+      <parameters>$(find rover_controller)/config/controller.yaml</parameters>
+    </plugin>
+  </gazebo>
+  <!-- Base -->
+  <xacro:gazebo_surface link_name="base_link" />
+  <!-- Wheels -->
+  <xacro:gazebo_surface link_name="wheel_back_left" />
+  <xacro:gazebo_surface link_name="wheel_front_left" />
+  <xacro:gazebo_surface link_name="wheel_back_right" />
+  <xacro:gazebo_surface link_name="wheel_front_right" />
+  <!-- Suspensions -->
+  <xacro:gazebo_surface link_name="suspension_right" />
+  <xacro:gazebo_surface link_name="suspension_left" />
 </robot>

File: src/rover_description/urdf/rover.material.xacro (robot description, xacro)
@@ -1,4 +1,10 @@
 <?xml version="1.0"?>
 <robot name="Deimos/material" xmlns:xacro="http://www.ros.org/wiki/xacro">
+  <material name="black">
+    <color rgba="0.01 0.01 0.01 1" />
+  </material>
+  <material name="white">
+    <color rgba="1 1 1 1" />
+  </material>
   <material name="silver">
     <color rgba="0.7 0.7 0.7 1" />
@@ -7,7 +13,4 @@
     <color rgba="0.12 0.18 0.4 1" />
   </material>
-  <material name="black">
-    <color rgba="0.01 0.01 0.01 1" />
-  </material>
   <material name="soft_orange">
     <color rgba="0.85 0.45 0.15 1" />

File: src/rover_description/urdf/rover.urdf.xacro (robot description, xacro)
@@ -1,8 +1,10 @@
 <?xml version="1.0"?>
 <robot name="Deimos" xmlns:xacro="http://www.ros.org/wiki/xacro">
-  <xacro:property name="PI" value="3.141592653589793"/>
+  <xacro:property name="PI" value="3.141592653589793" />
+  <xacro:property name="mesh_scale" value="0.001 0.001 0.001" />
   <xacro:include filename="$(find rover_description)/urdf/rover.material.xacro" />
   <xacro:include filename="$(find rover_description)/urdf/rover.gazebo.xacro" />
   <xacro:include filename="$(find rover_description)/urdf/sensors/lidar3d.xacro" />
+  <!-- <xacro:include filename="$(find rover_description)/urdf/rover.trans.xacro" /> -->
   <xacro:include filename="$(find rover_description)/urdf/rover.control.xacro" />
   <link name="base_footprint" />
@@ -10,10 +12,26 @@
     <parent link="base_footprint" />
     <child link="base_link" />
-    <origin xyz="0 0 0" rpy="0 0 ${PI/2}" />
-  </joint>
+    <origin xyz="-0.375 0.25 0" rpy="0 0 ${-PI/2}" />
+  </joint>
+  <joint name="lidar_joint" type="fixed">
+    <parent link="base_link" />
+    <child link="lidar_link" />
+    <origin xyz="0.25 0.8 0.1" rpy="0 0 0" />
+  </joint>
+  <link name="lidar_link">
+    <visual>
+      <origin xyz="0 0 0" rpy="0 0 0" />
+      <geometry>
+        <box size="0.05 0.05 0.05" />
+      </geometry>
+      <material name="dark">
+        <color rgba="0.1 0.1 0.1 1.0" />
+      </material>
+    </visual>
+  </link>
   <link name="base_link">
     <inertial>
       <origin xyz="0.23371470080552523 0.3424215459495483 0.11792924666461195" rpy="0 0 0" />
-      <mass value="360.0" />
+      <mass value="36.0" />
       <inertia ixx="28.457355" iyy="14.276737" izz="34.968035" ixy="0.085086" iyz="0.387247"
         ixz="-0.119086" />
@@ -24,7 +42,5 @@
         <mesh filename="package://rover_description/meshes/base_link.stl" scale="0.001 0.001 0.001" />
       </geometry>
-      <material name="nice_navy">
-        <color rgba="0.12 0.18 0.4 1" />
-      </material>
+      <material name="nice_navy" />
     </visual>
     <collision>
@@ -35,5 +51,5 @@
     </collision>
   </link>
-  <link name="Wheel2_1">
+  <link name="wheel_back_left">
     <inertial>
       <origin xyz="0.060000000000048695 9.626243984289795e-07 0.00010157518963996304" rpy="0 0 0" />
@@ -44,18 +60,18 @@
       <origin xyz="0.1758 0.049434 0.072191" rpy="0 0 0" />
       <geometry>
-        <mesh filename="package://rover_description/meshes/Wheel2_1.stl" scale="0.001 0.001 0.001" />
-      </geometry>
-      <material name="black">
-        <color rgba="0.01 0.01 0.01 1" />
-      </material>
+        <mesh filename="package://rover_description/meshes/wheel_back_left.stl"
+          scale="0.001 0.001 0.001" />
+      </geometry>
+      <material name="black" />
     </visual>
     <collision>
       <origin xyz="0.1758 0.049434 0.072191" rpy="0 0 0" />
       <geometry>
-        <mesh filename="package://rover_description/meshes/Wheel2_1.stl" scale="0.001 0.001 0.001" />
-      </geometry>
-    </collision>
-  </link>
-  <link name="Wheel1_1">
+        <mesh filename="package://rover_description/meshes/wheel_back_left.stl"
+          scale="0.001 0.001 0.001" />
+      </geometry>
+    </collision>
+  </link>
+  <link name="wheel_front_left">
     <inertial>
       <origin xyz="0.05999999999997653 1.1249441103089453e-06 0.00010186480729457159" rpy="0 0 0" />
@@ -66,18 +82,18 @@
       <origin xyz="0.1758 -0.800498 0.083039" rpy="0 0 0" />
       <geometry>
-        <mesh filename="package://rover_description/meshes/Wheel1_1.stl" scale="0.001 0.001 0.001" />
-      </geometry>
-      <material name="black">
-        <color rgba="0.01 0.01 0.01 1" />
-      </material>
+        <mesh filename="package://rover_description/meshes/wheel_front_left.stl"
+          scale="0.001 0.001 0.001" />
+      </geometry>
+      <material name="black" />
     </visual>
     <collision>
       <origin xyz="0.1758 -0.800498 0.083039" rpy="0 0 0" />
       <geometry>
-        <mesh filename="package://rover_description/meshes/Wheel1_1.stl" scale="0.001 0.001 0.001" />
-      </geometry>
-    </collision>
-  </link>
-  <link name="Wheel2__1__2">
+        <mesh filename="package://rover_description/meshes/wheel_front_left.stl"
+          scale="0.001 0.001 0.001" />
+      </geometry>
+    </collision>
+  </link>
+  <link name="wheel_back_right">
     <inertial>
       <origin xyz="-0.059999999999952314 1.1891813821787722e-06 0.00010132422446335054" rpy="0 0 0" />
@@ -88,44 +104,40 @@
       <origin xyz="-0.6425 0.049502 0.082708" rpy="0 0 0" />
       <geometry>
-        <mesh filename="package://rover_description/meshes/Wheel2__1__2.stl"
-          scale="0.001 0.001 0.001" />
-      </geometry>
-      <material name="black">
-        <color rgba="0.01 0.01 0.01 1" />
-      </material>
+        <mesh filename="package://rover_description/meshes/wheel_back_right.stl"
+          scale="0.001 0.001 0.001" />
+      </geometry>
+      <material name="black" />
     </visual>
     <collision>
       <origin xyz="-0.6425 0.049502 0.082708" rpy="0 0 0" />
       <geometry>
-        <mesh filename="package://rover_description/meshes/Wheel2__1__2.stl"
-          scale="0.001 0.001 0.001" />
-      </geometry>
-    </collision>
-  </link>
-  <link name="Wheel2__1__1">
-    <inertial>
-      <origin xyz="-0.7537999999999477 7.512494407269088e-05 0.00026586480728614525" rpy="0 0 0" />
+        <mesh filename="package://rover_description/meshes/wheel_back_right.stl"
+          scale="0.001 0.001 0.001" />
+      </geometry>
+    </collision>
+  </link>
+  <link name="wheel_front_right">
+    <inertial>
+      <origin xyz="-0.06 7.512494407269088e-05 0.00026586480728614525" rpy="0 0 0" />
       <mass value="35.0" />
       <inertia ixx="0.234154" iyy="0.134117" izz="0.153907" ixy="0.0" iyz="8e-06" ixz="-0.0" />
     </inertial>
     <visual>
-      <origin xyz="-1.3363 -0.800424 0.083203" rpy="0 0 0" />
-      <geometry>
-        <mesh filename="package://rover_description/meshes/Wheel2__1__1.stl"
-          scale="0.001 0.001 0.001" />
-      </geometry>
-      <material name="black">
-        <color rgba="0.01 0.01 0.01 1" />
-      </material>
-    </visual>
-    <collision>
-      <origin xyz="-1.3363 -0.800424 0.083203" rpy="0 0 0" />
-      <geometry>
-        <mesh filename="package://rover_description/meshes/Wheel2__1__1.stl"
-          scale="0.001 0.001 0.001" />
-      </geometry>
-    </collision>
-  </link>
-  <link name="Side1_1">
+      <origin xyz="-0.6425 -0.800424 0.083203" rpy="0 0 0" />
+      <geometry>
+        <mesh filename="package://rover_description/meshes/wheel_front_right.stl"
+          scale="0.001 0.001 0.001" />
+      </geometry>
+      <material name="black" />
+    </visual>
+    <collision>
+      <origin xyz="-0.6425 -0.800424 0.083203" rpy="0 0 0" />
+      <geometry>
+        <mesh filename="package://rover_description/meshes/wheel_front_right.stl"
+          scale="0.001 0.001 0.001" />
+      </geometry>
+    </collision>
+  </link>
+  <link name="suspension_right">
     <inertial>
       <origin xyz="-0.04997257661493937 0.0004804691908492642 0.02785086678998311" rpy="0 0 0" />
@@ -137,18 +149,18 @@
       <origin xyz="-0.63 -0.37785 -0.1081" rpy="0 0 0" />
       <geometry>
-        <mesh filename="package://rover_description/meshes/Side1_1.stl" scale="0.001 0.001 0.001" />
-      </geometry>
-      <material name="soft_orange">
-        <color rgba="0.85 0.45 0.15 1" />
-      </material>
+        <mesh filename="package://rover_description/meshes/suspension_right.stl"
+          scale="0.001 0.001 0.001" />
+      </geometry>
+      <material name="soft_orange" />
     </visual>
     <collision>
       <origin xyz="-0.63 -0.37785 -0.1081" rpy="0 0 0" />
       <geometry>
-        <mesh filename="package://rover_description/meshes/Side1_1.stl" scale="0.001 0.001 0.001" />
-      </geometry>
-    </collision>
-  </link>
-  <link name="Side2_1">
+        <mesh filename="package://rover_description/meshes/suspension_right.stl"
+          scale="0.001 0.001 0.001" />
+      </geometry>
+    </collision>
+  </link>
+  <link name="suspension_left">
     <inertial>
       <origin xyz="0.050023043717073556 0.00048164194190997156 0.028033001206298203" rpy="0 0 0" />
@@ -160,51 +172,51 @@
       <origin xyz="0.1638 -0.37785 -0.1081" rpy="0 0 0" />
       <geometry>
-        <mesh filename="package://rover_description/meshes/Side2_1.stl" scale="0.001 0.001 0.001" />
-      </geometry>
-      <material name="soft_orange">
-        <color rgba="0.85 0.45 0.15 1" />
-      </material>
+        <mesh filename="package://rover_description/meshes/suspension_left.stl"
+          scale="0.001 0.001 0.001" />
+      </geometry>
+      <material name="soft_orange" />
     </visual>
     <collision>
       <origin xyz="0.1638 -0.37785 -0.1081" rpy="0 0 0" />
       <geometry>
-        <mesh filename="package://rover_description/meshes/Side2_1.stl" scale="0.001 0.001 0.001" />
-      </geometry>
-    </collision>
-  </link>
-  <joint name="Revolute 14" type="continuous">
+        <mesh filename="package://rover_description/meshes/suspension_left.stl"
+          scale="0.001 0.001 0.001" />
+      </geometry>
+    </collision>
+  </link>
+  <joint name="wheel_back_left_joint" type="continuous">
     <origin xyz="-0.012 -0.427284 -0.180291" rpy="0 0 0" />
-    <parent link="Side2_1" />
-    <child link="Wheel2_1" />
-    <axis xyz="-1.0 0.0 -0.0" />
-  </joint>
-  <joint name="Revolute 15" type="continuous">
+    <parent link="suspension_left" />
+    <child link="wheel_back_left" />
+    <axis xyz="-1 0 0" />
+  </joint>
+  <joint name="wheel_front_left_joint" type="continuous">
     <origin xyz="-0.012 0.422648 -0.191139" rpy="0 0 0" />
-    <parent link="Side2_1" />
-    <child link="Wheel1_1" />
-    <axis xyz="-1.0 0.0 -0.0" />
-  </joint>
-  <joint name="Revolute 16" type="continuous">
+    <parent link="suspension_left" />
+    <child link="wheel_front_left" />
+    <axis xyz="-1 0 0" />
+  </joint>
+  <joint name="wheel_back_right_joint" type="continuous">
     <origin xyz="0.0125 -0.427352 -0.190808" rpy="0 0 0" />
-    <parent link="Side1_1" />
-    <child link="Wheel2__1__2" />
-    <axis xyz="1.0 -0.0 0.0" />
-  </joint>
-  <joint name="Revolute 17" type="continuous">
-    <origin xyz="0.7063 0.422574 -0.191303" rpy="0 0 0" />
-    <parent link="Side1_1" />
-    <child link="Wheel2__1__1" />
-    <axis xyz="1.0 -0.0 0.0" />
-  </joint>
-  <joint name="Revolute 18" type="fixed">
+    <parent link="suspension_right" />
+    <child link="wheel_back_right" />
+    <axis xyz="-1 0 0" />
+  </joint>
+  <joint name="wheel_front_right_joint" type="continuous">
+    <origin xyz="0.0125 0.422574 -0.191303" rpy="0 0 0" />
+    <parent link="suspension_right" />
+    <child link="wheel_front_right" />
+    <axis xyz="-1 0 0" />
+  </joint>
+  <joint name="suspension_right_joint" type="fixed">
     <origin xyz="0.63 0.37785 0.1081" rpy="0 0 0" />
     <parent link="base_link" />
-    <child link="Side1_1" />
+    <child link="suspension_right" />
     <axis xyz="1.0 -0.0 0.0" />
   </joint>
-  <joint name="Revolute 19" type="fixed">
+  <joint name="suspension_left_joint" type="fixed">
     <origin xyz="-0.1638 0.37785 0.1081" rpy="0 0 0" />
     <parent link="base_link" />
-    <child link="Side2_1" />
+    <child link="suspension_left" />
     <axis xyz="-1.0 0.0 -0.0" />
   </joint>

File: src/rover_description/urdf/sensors/lidar3d.xacro (robot description, xacro)
@@ -1,20 +1,4 @@
 <?xml version="1.0"?>
 <robot xmlns:xacro="http://ros.org/wiki/xacro">
-  <joint name="lidar_joint" type="fixed">
-    <parent link="base_link" />
-    <child link="lidar_link" />
-    <origin xyz="0.0 0.0 0.25" rpy="0 0 0" />
-  </joint>
-  <link name="lidar_link">
-    <visual>
-      <origin xyz="0 0 0" rpy="0 0 0" />
-      <geometry>
-        <box size="0.1 0.1 0.05" />
-      </geometry>
-      <material name="dark">
-        <color rgba="0.1 0.1 0.1 1.0" />
-      </material>
-    </visual>
-  </link>
   <gazebo reference="lidar_link">
     <sensor name="lidar3d" type="gpu_lidar">
@@ -41,5 +25,5 @@
         </scan>
         <range>
-          <min>0.20</min>
+          <min>0.50</min>
           <max>50.0</max>
           <resolution>0.01</resolution>
