Commit message: Select ros2_control hardware plugin by ROS distro
Agent-Logs-Url: https://github.com/SheffMarsworks/DeimosRover-2025-2026-/sessions/0bb9b9a4-d164-429e-83d5-a08a56300289

Co-authored-by: TanukiDong <85825293+TanukiDong@users.noreply.github.com>

File: src/rover_description/urdf/rover.control.xacro (robot description, xacro)
@@ -14,6 +14,11 @@
   </xacro:macro>
   <ros2_control name="GazeboSystem" type="system">
+    <xacro:property name="ros_distro" value="$(env ROS_DISTRO humble)" />
+    <xacro:property
+      name="ros2_control_system_plugin"
+      value="${'ign_ros2_control/IgnitionSystem' if ros_distro == 'humble' else 'gz_ros2_control/GazeboSimSystem'}" />
     <hardware>
-      <plugin>ign_ros2_control/IgnitionSystem</plugin>
+      <!-- <plugin>ign_ros2_control/IgnitionSystem</plugin> -->
+      <plugin>${ros2_control_system_plugin}</plugin>
     </hardware>
     <xacro:wheel_ros2_control_joint joint_name="wheel_back_left_joint" />
