Commit message: fix

File: src/rover_description/urdf/rover.gazebo.xacro (robot description, xacro)
@@ -1,5 +1,4 @@
 <?xml version="1.0"?>
 <robot name="Deimos_Gazebo" xmlns:xacro="http://www.ros.org/wiki/xacro">
-  <xacro:property name="body_color" value="Gazebo/Silver" />
   <xacro:property name="default_mu1" value="0.2" />
   <xacro:property name="default_mu2" value="0.2" />

File: src/rover_description/urdf/sensors/lidar3d.xacro (robot description, xacro)
@@ -12,5 +12,5 @@
         <scan>
           <horizontal>
-            <samples>1024</samples>
+            <samples>512</samples>
             <resolution>1</resolution>
             <min_angle>${-PI/2}</min_angle>
