Commit message: change name body_link → base_link

File: src/rover_description/urdf/rover.urdf.xacro (robot description, xacro)
@@ -12,9 +12,9 @@
     <joint name="base_footprint_joint" type="fixed">
         <parent link="base_footprint"/>
-        <child link="body_link"/>
+        <child link="base_link"/>
         <origin xyz="0 0 0.393" rpy="0 0 0"/>
     </joint>
     <!-- This is the body of the rover -->
-    <link name="body_link">
+    <link name="base_link">
         <inertial>
             <origin xyz="0 0 0" rpy="0 0 0"/>
@@ -41,5 +41,5 @@
     <!-- This is the left suspension assembly -->
     <joint name="susLeft_joint" type="fixed">
-        <parent link="body_link" />
+        <parent link="base_link" />
         <child link="susLeft_link" />
         <origin xyz ="-0.1 -0.239 0.04" rpy="0 0 -1.579795" />
@@ -100,5 +100,5 @@
     <!-- This is the right suspension assembly -->
     <joint name="susRight_joint" type="fixed">
-        <parent link="body_link" />
+        <parent link="base_link" />
         <child link="susRight_link" />
         <origin xyz ="-0.1 0.21 0.04" rpy="0 0 -1.579795" />
@@ -333,5 +333,5 @@
     <!-- This is the back left wheel of the rover
     <joint name="wheel2_joint" type="continuous">
-        <parent link="body_link" />
+        <parent link="base_link" />
         <child link="wheel2_link" />
         <origin xyz ="-0.3 0.35 -0.1" rpy="0 0 0" />

File: src/rover_description/urdf/sensors/lidar3d.xacro (robot description, xacro)
@@ -2,5 +2,5 @@
 <robot xmlns:xacro="http://ros.org/wiki/xacro">
   <joint name="lidar_joint" type="fixed">
-    <parent link="body_link" />
+    <parent link="base_link" />
     <child link="lidar_link" />
     <origin xyz="0.0 0.0 0.25" rpy="0 0 0" />

File: src/rover_description/urdf/sensors/realsense.xacro (robot description, xacro)
@@ -3,5 +3,5 @@
   <xacro:property name="PI" value="3.14159265"/>
   <joint name="realsense_joint" type="fixed">
-    <parent link="body_link"/>
+    <parent link="base_link"/>
     <child link="realsense_link"/>
     <origin xyz="-0.39 0.0 0.08" rpy="0.0 0.0 ${pi}"/>

Commit message: fix/temporary rotate rover to match odom

File: src/rover_description/urdf/rover.urdf.xacro (robot description, xacro)
@@ -13,5 +13,5 @@
         <parent link="base_footprint"/>
         <child link="base_link"/>
-        <origin xyz="0 0 0.393" rpy="0 0 0"/>
+        <origin xyz="0 0 0.393" rpy="0 0 3.14159"/>
     </joint>
     <!-- This is the body of the rover -->

Commit message: refactor code

File: src/rover_description/urdf/rover.urdf.xacro (robot description, xacro)
@@ -12,5 +12,5 @@
     <parent link="base_footprint" />
     <child link="base_link" />
-    <origin xyz="-0.375 0.25 0" rpy="0 0 ${-PI/2}" />
+    <origin xyz="-0.375 0.235 0.222" rpy="0 0 ${-PI/2}" />
   </joint>
   <joint name="lidar_joint" type="fixed">
@@ -30,4 +30,5 @@
     </visual>
   </link>
+  <!-- Chassis is 752 x 470 x 222 mm -->
   <link name="base_link">
     <inertial>

Commit message: re-add depth camera

File: src/rover_description/urdf/rover.urdf.xacro (robot description, xacro)
@@ -8,4 +8,5 @@
   <!-- <xacro:include filename="$(find rover_description)/urdf/rover.trans.xacro" /> -->
   <xacro:include filename="$(find rover_description)/urdf/rover.control.xacro" />
+  <xacro:include filename="$(find rover_description)/urdf/sensors/realsense.xacro" />
   <link name="base_footprint" />
   <joint name="base_footprint_joint" type="fixed">
@@ -14,8 +15,13 @@
     <origin xyz="-0.375 0.235 0.222" rpy="0 0 ${-PI/2}" />
   </joint>
+  <joint name="realsense_joint" type="fixed">
+    <parent link="base_link" />
+    <child link="realsense_link" />
+    <origin xyz="0.25 0.8 0.15" rpy="0.0 0.0 ${PI/2}" />
+  </joint>
   <joint name="lidar_joint" type="fixed">
     <parent link="base_link" />
     <child link="lidar_link" />
-    <origin xyz="0.25 0.8 0.1" rpy="0 0 0" />
+    <origin xyz="0.25 0.75 0.1" rpy="0 0 0" />
   </joint>
   <link name="lidar_link">
@@ -55,5 +61,5 @@
     <inertial>
       <origin xyz="0.060000000000048695 9.626243984289795e-07 0.00010157518963996304" rpy="0 0 0" />
-      <mass value="35.0" />
+      <mass value="100.0" />
       <inertia ixx="0.234154" iyy="0.134117" izz="0.153907" ixy="-0.0" iyz="8e-06" ixz="0.0" />
     </inertial>

Commit message: Update Livox LiDAR model

File: src/rover_description/urdf/rover.urdf.xacro (robot description, xacro)
@@ -12,16 +12,17 @@
     <origin xyz="0 0 0.2" rpy="0 0 0" />
   </joint>
-  <joint name="lidar_joint" type="fixed">
+  <joint name="livox_joint" type="fixed">
     <parent link="base_link" />
-    <child link="lidar_link" />
+    <child link="livox_frame" />
+    <!-- Change transform to the actual position -->
     <origin xyz="0.5 0 0.1" rpy="0 0 0" />
   </joint>
-  <link name="lidar_link">
-    <visual>
-      <origin xyz="0 0 0" rpy="0 0 0" />
-      <geometry>
-        <box size="0.05 0.05 0.05" />
-      </geometry>
-      <material name="black" />
+  <link name="livox_frame">
+    <visual>
+      <origin xyz="0 0 0" rpy="${PI/2} 0 0" />
+      <geometry>
+        <mesh filename="package://rover_description/meshes/livox-mid-360.stl" scale="0.001 0.001 0.001" />
+      </geometry>
+      <material name="white" />
     </visual>
   </link>
